File: kicad/remote.sch (KiCad schematic (older format))
At the start: 27 parts

Commit message: Update diagram.
Parts:
- removed C?: C, symbol C
- removed R? (x10): R, symbol R
- removed SW? (x4): SW_Push, symbol SW_Push
- removed SW? (x4): SW_SPST, symbol SW_SPST
- removed U?: Arduino_Micro, symbol Arduino_Micro
- removed U?: Adafruit_SSD1306, symbol Adafruit_SSD1306
- added C? (x3): C, symbol C
- added P1: Left joystick, symbol POT_Dual_Separate
- added P2 (x2): Right joystick, symbol POT_Dual_Separate
- added U?: OLED_7pin_4SPI, symbol OLED_7pin_4SPI
- added U?: arduino_mini, DIL20, symbol arduino_mini
- added U?: AP1117, TO_SOT_Packages_SMD:SOT-223, symbol AP1117
Connections:
- net labels added: +3V3, A4, A5, A6, A7, D10, D9
- wire segments 87 -> 104
- no-connect marks 2 -> 6
Other:
- moved on the sheet: U?
