File: kicad/remote.sch (KiCad schematic (older format))
At the start: 15 parts, among them P1 Left joystick, P2 Right joystick

Commit message: Prepare for PCB.
Parts:
- removed C? (x3): C, symbol C
- removed P1: Left joystick, symbol POT_Dual_Separate
- removed P2 (x2): Right joystick, symbol POT_Dual_Separate
- removed U?: arduino_mini, DIL20, symbol arduino_mini
- added C4: 22u, Capacitor_SMD:C_1206_3216Metric, symbol Device:CP
- added C5: 1u, Capacitor_SMD:C_0805_2012Metric, symbol Device:C
- added H1, H2, H3, H4: MountingHole, MountingHole:MountingHole_3.2mm_M3, symbol Mechanical:MountingHole
- added J1: Conn_01x03, Connector_JST:JST_XH_B03B-XH-A_1x03_P2.50mm_Vertical, symbol Connector_Generic:Conn_01x03
- added U3: Arduino_Nano_v3.x, Module:Arduino_Nano, symbol MCU_Module:Arduino_Nano_v3.x
- added U7, U8: COM-09032, Remote:XDCR_COM-09032, symbol COM-09032:COM-09032
- C1, C2, C3: renamed from C?; value C -> 1u; footprint (none) -> Capacitor_SMD:C_0805_2012Metric; symbol C -> remote-rescue:C
- RV1, RV2: renamed from RV?; footprint (none) -> Remote:Switch_1x03_P5.08mm; symbol POT -> remote-rescue:POT
- U4: renamed from U?; footprint TO_SOT_Packages_SMD:SOT-223 -> Package_TO_SOT_SMD:SOT-223; symbol AP1117 -> remote-rescue:AP1117
- U5: renamed from U?; footprint MODULE -> Remote:nRF24L01; symbol nRF24L01+ -> remote-rescue:nRF24L01+
- U6: renamed from U?; footprint (none) -> Remote:Display_OLED_7pin_4SPI; symbol OLED_7pin_4SPI -> remote-rescue:OLED_7pin_4SPI
Connections:
- net +3V3: now also C4.1, C5.2
- net +5V: now also J1.1 (Pin_1), U3.27 (+5V), U7.H1 (H+), U7.V1 (V+), U8.H1 (H+), U8.V1 (V+)
- net A4: now also J1.2 (Pin_2), U3.23 (A4)
- net A6: now also U3.25 (A6)
- net A7: now also U3.26 (A7)
- net GND: now also C4.2, C5.1, J1.3 (Pin_3), U3.29 (GND), U3.4 (GND), U7.H3 (H-), U7.S1 (SHIELD), U7.S2 (SHIELD), U7.S3 (SHIELD), U7.S4 (SHIELD), U7.V3 (V-), U8.H3 (H-), U8.S1 (SHIELD), U8.S2 (SHIELD), U8.S3 (SHIELD), U8.S4 (SHIELD), U8.V3 (V-)
- net CE: now reaches U5.3 (CE)
- net CE: now also U3.10 (D7)
- net CSN: now reaches U5.4 (CSN)
- net CSN: now also U3.11 (D8)
- net SCK: now reaches U5.5 (SCK)
- net SCK: now also U6.3 (SCK), U3.16 (D13), U3.9 (D6)
- net MOSI: now reaches U5.6 (MOSI)
- net MOSI: now also U3.14 (D11)
- net MISO: now reaches U5.7 (MISO)
- net MISO: now also U3.15 (D12)
- net SDA: now reaches U6.4 (SDA)
- net SDA: now also U3.8 (D5)
- net RESET: now reaches U6.5 (RES)
- net RESET: now also U3.7 (D4)
- net DC: now reaches U6.6 (DC)
- net DC: now also U3.6 (D3)
- net CS: now reaches U6.7 (CS)
- net CS: now also U3.5 (D2)
- new net: U3.19 (A0), U7.V2 (V)
- new net: U3.20 (A1), U7.H2 (H)
- new net: U3.21 (A2), U8.V2 (V)
- new net: U3.22 (A3), U8.H2 (H)
- new net CP: U3.12 (D9)
- new net PL: U3.24 (A5)
- new net Q7: U3.13 (D10)
- no-connect marks 6 -> 12
Other:
- note added: "+5V IN"
- note added: "BATT SENSE"
- note added: "GND"
- moved on the sheet: C2

Commit message: Add more switches, footprints.
Parts:
- J1: footprint Connector_JST:JST_XH_B03B-XH-A_1x03_P2.50mm_Vertical -> Milling:JST_XH_B03B-XH-A_1x03_P2.50mm_Vertical_Milling
- RV1, RV2: footprint Remote:Switch_1x03_P5.08mm -> Remote:Potentiometer_4mm_axis
Changed lines of the file:
@@
 F 0 "RV1" V 6825 3600 50  0000 C CNN
 F 1 "POT" V 6900 3600 50  0000 C CNN
-F 2 "Remote:Switch_1x03_P5.08mm" H 7000 3600 50  0001 C CNN
+F 2 "Remote:Potentiometer_4mm_axis" H 7000 3600 50  0001 C CNN
 F 3 "" H 7000 3600 50  0001 C CNN
 	1    7000 3600
@@
 F 0 "RV2" V 7875 3600 50  0000 C CNN
 F 1 "POT" V 7950 3600 50  0000 C CNN
-F 2 "Remote:Switch_1x03_P5.08mm" H 8050 3600 50  0001 C CNN
+F 2 "Remote:Potentiometer_4mm_axis" H 8050 3600 50  0001 C CNN
 F 3 "" H 8050 3600 50  0001 C CNN
 	1    8050 3600
@@
 F 0 "J1" H 1068 1667 50  0000 C CNN
 F 1 "Conn_01x03" H 1068 1576 50  0000 C CNN
-F 2 "Connector_JST:JST_XH_B03B-XH-A_1x03_P2.50mm_Vertical" H 1150 1350 50  0001 C CNN
+F 2 "Milling:JST_XH_B03B-XH-A_1x03_P2.50mm_Vertical_Milling" H 1150 1350 50  0001 C CNN
 F 3 "~" H 1150 1350 50  0001 C CNN
 	1    1150 1350

Commit message: Place switches, etc. Split up into two boards.
Parts:
- added J2, J6: Conn_01x02, Milling:JST_XH_B02B-XH-A_1x02_P2.50mm_Vertical_Milling, symbol Connector_Generic:Conn_01x02
- added J3: Conn_01x07, Connector_JST:JST_XH_B07B-XH-A_1x07_P2.50mm_Vertical, symbol Connector_Generic:Conn_01x07
- added J4, J5, J7: Conn_01x03, Milling:JST_XH_B03B-XH-A_1x03_P2.50mm_Vertical_Milling, symbol Connector_Generic:Conn_01x03
Connections:
- net +5V: now also J4.1 (Pin_1), J5.1 (Pin_1)
- net A4: now also RV1.2, J7.1 (Pin_1); no longer J1.2 (Pin_2), U3.23 (A4)
- net A6: now also RV2.2, J7.3 (Pin_3); no longer RV1.2, U3.25 (A6)
- net GND: now also J4.3 (Pin_3), J5.3 (Pin_3)
- net PL: now also U3.26 (A7); no longer U3.24 (A5)
- net at U3.19 (A0): now also J3.1 (Pin_1); no longer U7.V2 (V)
- net at U3.20 (A1): now also J3.2 (Pin_2); no longer U7.H2 (H)
- net at U3.21 (A2): now also J3.3 (Pin_3); no longer U8.V2 (V)
- net at U3.22 (A3): now also J3.4 (Pin_4); no longer U8.H2 (H)
- removed net A7: RV2.2, U3.26 (A7)
- new net: J3.5 (Pin_5), U3.23 (A4)
- new net: J3.6 (Pin_6), U3.24 (A5)
- new net: J3.7 (Pin_7), U3.25 (A6)
- new net: J6.2 (Pin_2), U7.H2 (H)
- new net: J6.1 (Pin_1), U7.V2 (V)
- new net: J2.2 (Pin_2), U8.H2 (H)
- new net: J2.1 (Pin_1), U8.V2 (V)
- new net A5: J5.2 (Pin_2), J7.2 (Pin_2)
- new net BAT: J1.2 (Pin_2), J4.2 (Pin_2)
Other:
- moved on the sheet: C3, C4, C5, H1, H2, H3, H4, RV1, RV2, U4, U5
