File: mainboard/switches.sch (KiCad schematic (older format))
At the start: 32 parts, among them J10 Conn_01x03, J11 Conn_01x03, J12 Conn_01x02, J13 Conn_01x04, J14 Conn_01x04, SW1 SW_SPDT_MSM, SW10 SW_Push, SW11 SW_DP3T, SW2 SW_SPDT_MSM, SW3 SW_SPDT_MSM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

Commit message: Update for I2C display.
Changed lines of the file:
@@
 	0    1    1    0
 $EndComp
-Text GLabel 5100 2600 0    60   Input ~ 0
-CP
-Text GLabel 5100 2450 0    60   Input ~ 0
-PL
 $Comp
 L remote-rescue:SW_Push SW10
