File: controller/switches.kicad_sch (KiCad schematic)
At the start: 6 parts, among them J8 Conn_01x08, J9 Conn_01x08, U1 74HC165, U2 74HC165

Commit message: Add debug connector.
Connections:
- net +5V renamed +3V3
Other:
- moved on the sheet: J8, U2

Commit message: Add switches, regulator, etc.
Parts:
- renumbered J8 to J4, J9 to J5
