File: mainboard-split/remote.kicad_pcb (KiCad board)
At the start: 2 copper layers, 171.7 x 109 mm, 22 parts, among them J1 Conn_01x02, J2 Conn_01x04, J3 Conn_01x03, J4 Conn_01x02, SW1 SW_SPDT_MSM, SW2 SW_SPDT_MSM, SW3 SW_Push, SW4 SW_Push, SW5 SW_Push

Commit message: Add more power.
Parts:
- added J5: 3V3 OUT, Connector_JST:JST_XH_B02B-XH-A_1x02_P2.50mm_Vertical, F.Cu at (134.9, 155.2)
- added J6: STICK POWER, Connector_JST:JST_XH_B02B-XH-A_1x02_P2.50mm_Vertical, F.Cu at (134.9, 163.0)
- J1: value Conn_01x02 -> 3V3 IN
