File: mainboard-split/mainboard.kicad_sch (KiCad schematic)
At the start: 24 parts, among them J1 3V3 IN, J2 Conn_01x04, J3 Conn_01x03, J4 Conn_01x02, J5 3V3 OUT, J6 STICK POWER, SW1 SW_SPDT_MSM, SW2 SW_SPDT_MSM, SW3 SW_Push, SW4 SW_Push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

Commit message: Rename project.
Parts:
- R5, R6, R7: symbol remote-rescue:R -> mainboard-rescue:R
- RV1: symbol remote-rescue:POT -> mainboard-rescue:POT
- SW1, SW2: symbol remote-rescue:SW_SPDT_MSM -> mainboard-rescue:SW_SPDT_MSM
- SW3, SW4, SW5: symbol remote-rescue:SW_Push -> mainboard-rescue:SW_Push
Changed lines of the file:
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@@
 	)
 	(symbol
-		(lib_id "remote-rescue:POT")
+		(lib_id "mainboard-rescue:POT")
 		(at 196.85 35.56 0)
 		(mirror y)
@@
 		)
 		(instances
-			(project "remote"
+			(project "mainboard"
 				(path "/1165cfa6-851c-4b44-8eb4-6a1ddaec09fb"
 					(reference "RV1")
@@
 	)
 	(symbol
-		(lib_id "remote-rescue:GND")
+		(lib_id "mainboard-rescue:GND")
 		(at 196.85 48.26 0)
 		(unit 1)
@@
 		)
 		(instances
-			(project "remote"
+			(project "mainboard"
 				(path "/1165cfa6-851c-4b44-8eb4-6a1ddaec09fb"
 					(reference "#PWR0104")
@@
 	)
 	(symbol
-		(lib_id "remote-rescue:+5V")
+		(lib_id "mainboard-rescue:+5V")
 		(at 196.85 22.86 0)
 		(unit 1)
@@
 		)
 		(instances
-			(project "remote"
+			(project "mainboard"
 				(path "/1165cfa6-851c-4b44-8eb4-6a1ddaec09fb"
 					(reference "#PWR0105")
@@
 		)
 		(instances
-			(project "remote"
+			(project "mainboard"
 				(path "/1165cfa6-851c-4b44-8eb4-6a1ddaec09fb"
 					(reference "#PWR0109")
@@
 		)
 		(instances
-			(project "remote"
+			(project "mainboard"
 				(path "/1165cfa6-851c-4b44-8eb4-6a1ddaec09fb"
 					(reference "#PWR0111")
@@
 		)
 		(instances
-			(project "remote"
+			(project "mainboard"
 				(path "/1165cfa6-851c-4b44-8eb4-6a1ddaec09fb"
 					(reference "#FLG0101")
@@
 		)
 		(instances
-			(project "remote"
+			(project "mainboard"
 				(path "/1165cfa6-851c-4b44-8eb4-6a1ddaec09fb"
 					(reference "#PWR0127")
@@
 		)
 		(instances
-			(project "remote"
+			(project "mainboard"
 				(path "/1165cfa6-851c-4b44-8eb4-6a1ddaec09fb"
 					(reference "#FLG0102")
@@
 		)
 		(instances
-			(project "remote"
+			(project "mainboard"
 				(path "/1165cfa6-851c-4b44-8eb4-6a1ddaec09fb"
 					(reference "#PWR0128")
@@
 		)
 		(instances
-			(project "remote"
+			(project "mainboard"
 				(path "/1165cfa6-851c-4b44-8eb4-6a1ddaec09fb"
 					(reference "J1")
@@
 		)
 		(instances
-			(project "remote"
+			(project "mainboard"
 				(path "/1165cfa6-851c-4b44-8eb4-6a1ddaec09fb"
 					(reference "J4")
@@
 		)
 		(instances
-			(project "remote"
+			(project "mainboard"
 				(path "/1165cfa6-851c-4b44-8eb4-6a1ddaec09fb"
 					(reference "H1")
@@
 		)
 		(instances
-			(project "remote"
+			(project "mainboard"
 				(path "/1165cfa6-851c-4b44-8eb4-6a1ddaec09fb"
 					(reference "H2")
@@
 		)
 		(instances
-			(project "remote"
+			(project "mainboard"
 				(path "/1165cfa6-851c-4b44-8eb4-6a1ddaec09fb"
 					(reference "H3")
@@
 		)
 		(instances
-			(project "remote"
+			(project "mainboard"
 				(path "/1165cfa6-851c-4b44-8eb4-6a1ddaec09fb"
 					(reference "H4")
@@
 	)
 	(symbol
-		(lib_id "remote-rescue:+5V")
+		(lib_id "mainboard-rescue:+5V")
 		(at 147.32 77.47 0)
 		(unit 1)
@@
 		)
 		(instances
-			(project "remote"
+			(project "mainboard"
 				(path "/1165cfa6-851c-4b44-8eb4-6a1ddaec09fb"
 					(reference "#PWR05")
@@
 	)
 	(symbol
-		(lib_id "remote-rescue:SW_Push")
+		(lib_id "mainboard-rescue:SW_Push")
 		(at 147.32 119.38 270)
 		(unit 1)
@@
 		)
 		(instances
-			(project "remote"
+			(project "mainboard"
 				(path "/1165cfa6-851c-4b44-8eb4-6a1ddaec09fb"
 					(reference "SW3")
@@
 	)
 	(symbol
-		(lib_id "remote-rescue:SW_SPDT_MSM")
+		(lib_id "mainboard-rescue:SW_SPDT_MSM")
 		(at 52.07 114.3 90)
 		(unit 1)
@@
 		)
 		(instances
-			(project "remote"
+			(project "mainboard"
 				(path "/1165cfa6-851c-4b44-8eb4-6a1ddaec09fb"
 					(reference "SW2")
@@
 	)
 	(symbol
-		(lib_id "remote-rescue:SW_SPDT_MSM")
+		(lib_id "mainboard-rescue:SW_SPDT_MSM")
 		(at 39.37 114.3 90)
 		(unit 1)
@@
 		)
 		(instances
-			(project "remote"
+			(project "mainboard"
 				(path "/1165cfa6-851c-4b44-8eb4-6a1ddaec09fb"
 					(reference "SW1")
@@
 		)
 		(instances
-			(project "remote"
+			(project "mainboard"
 				(path "/1165cfa6-851c-4b44-8eb4-6a1ddaec09fb"
 					(reference "R1")
@@
 		)
 		(instances
-			(project "remote"
+			(project "mainboard"
 				(path "/1165cfa6-851c-4b44-8eb4-6a1ddaec09fb"
 					(reference "J2")
@@
 		)
 		(instances
-			(project "remote"
+			(project "mainboard"
 				(path "/1165cfa6-851c-4b44-8eb4-6a1ddaec09fb"
 					(reference "R2")
@@
 		)
 		(instances
-			(project "remote"
+			(project "mainboard"
 				(path "/1165cfa6-851c-4b44-8eb4-6a1ddaec09fb"
 					(reference "J3")
@@
 	)
 	(symbol
-		(lib_id "remote-rescue:GND")
+		(lib_id "mainboard-rescue:GND")
 		(at 147.32 129.54 0)
 		(unit 1)
@@
 		)
 		(instances
-			(project "remote"
+			(project "mainboard"
 				(path "/1165cfa6-851c-4b44-8eb4-6a1ddaec09fb"
 					(reference "#PWR06")
@@
 		)
 		(instances
-			(project "remote"
+			(project "mainboard"
 				(path "/1165cfa6-851c-4b44-8eb4-6a1ddaec09fb"
 					(reference "R3")
@@
 		)
 		(instances
-			(project "remote"
+			(project "mainboard"
 				(path "/1165cfa6-851c-4b44-8eb4-6a1ddaec09fb"
 					(reference "#PWR04")
@@
 	)
 	(symbol
-		(lib_id "remote-rescue:R")
+		(lib_id "mainboard-rescue:R")
 		(at 147.32 88.9 0)
 		(unit 1)
@@
 		)
 		(instances
-			(project "remote"
+			(project "mainboard"
 				(path "/1165cfa6-851c-4b44-8eb4-6a1ddaec09fb"
 					(reference "R5")
@@
 		)
 		(instances
-			(project "remote"
+			(project "mainboard"
 				(path "/1165cfa6-851c-4b44-8eb4-6a1ddaec09fb"
 					(reference "#PWR03")
@@
 	)
 	(symbol
-		(lib_id "remote-rescue:SW_Push")
+		(lib_id "mainboard-rescue:SW_Push")
 		(at 170.18 119.38 270)
 		(unit 1)
@@
 		)
 		(instances
-			(project "remote"
+			(project "mainboard"
 				(path "/1165cfa6-851c-4b44-8eb4-6a1ddaec09fb"
 					(reference "SW5")
@@
 	)
 	(symbol
-		(lib_id "remote-rescue:R")
+		(lib_id "mainboard-rescue:R")
 		(at 170.18 88.9 0)
 		(unit 1)
@@
 		)
 		(instances
-			(project "remote"
+			(project "mainboard"
 				(path "/1165cfa6-851c-4b44-8eb4-6a1ddaec09fb"
 					(reference "R7")
@@
 	)
 	(symbol
-		(lib_id "remote-rescue:SW_Push")
+		(lib_id "mainboard-rescue:SW_Push")
 		(at 158.75 119.38 270)
 		(unit 1)
@@
 		)
 		(instances
-			(project "remote"
+			(project "mainboard"
 				(path "/1165cfa6-851c-4b44-8eb4-6a1ddaec09fb"
 					(reference "SW4")
@@
 		)
 		(instances
-			(project "remote"
+			(project "mainboard"
 				(path "/1165cfa6-851c-4b44-8eb4-6a1ddaec09fb"
 					(reference "R4")
@@
 	)
 	(symbol
-		(lib_id "remote-rescue:R")
+		(lib_id "mainboard-rescue:R")
 		(at 158.75 88.9 0)
 		(unit 1)
@@
 		)
 		(instances
-			(project "remote"
+			(project "mainboard"
 				(path "/1165cfa6-851c-4b44-8eb4-6a1ddaec09fb"
 					(reference "R6")
