File: mainboard-split/mainboard.kicad_pcb (KiCad board)
At the start: 2 copper layers, 49.7 x 83.3 mm, 24 parts, among them J1 3V3 IN, J2 Conn_01x04, J3 Conn_01x03, J4 Conn_01x02, J5 3V3 OUT, J6 STICK POWER, SW1 SW_SPDT_MSM, SW2 SW_SPDT_MSM, SW3 SW_Push, SW4 SW_Push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

Commit message: Use Vref for pots and sticks.
Parts:
- J1: value 3V3 IN -> Vbat in
- J5: value 3V3 OUT -> Vbat out
- J6: value STICK POWER -> Vref in
- moved J6 34.1 mm to (71.0, 191.2)
- moved J3 2.24 mm to (64.0, 185.4)
Connections:
- net A7 renamed Net-(J4-Pin_1)
- C1 pad 1: +3V3 -> +2V5
- J4 pad 2: unconnected-(J4-Pin_2-Pad2) -> +2V5
- J6 pad 1: +3V3 -> +2V5
- RV1 pad 1: +3V3 -> +2V5
Routing:
- net GND: track 159.4 -> 195.9 mm
- net +2V5: track 0.00 -> 15.1 mm
- net +3V3: track 137.8 -> 125.5 mm, vias 1 -> 3
- net Net-(J3-Pin_2): track 19.6 -> 17.9 mm
- net Net-(J3-Pin_1): track 31.9 -> 31.0 mm
- net Net-(J3-Pin_3): track 36.4 -> 35.5 mm
